Commit message: working gps/motor/compass

File: install/tractor_bringup/share/tractor_bringup/urdf/tractor.urdf.xacro (robot description, xacro)
@@ -3,11 +3,15 @@
   <!-- Properties -->
   <xacro:property name="PI" value="3.14159"/>
-  <xacro:property name="wheel_radius" value="0.15"/>
-  <xacro:property name="wheel_width" value="0.25"/>
-  <xacro:property name="wheel_separation" value="0.7"/>
-  <xacro:property name="track_length" value="0.6"/>
-  <xacro:property name="base_length" value="0.8"/>
-  <xacro:property name="base_width" value="0.6"/>
-  <xacro:property name="base_height" value="0.3"/>
+  <!-- Robot dimensions based on actual measurements -->
+  <!-- Main body: 102mm wide × 266.7mm long × 90mm height -->
+  <!-- Treads: 42mm wide each, same length and height as body -->
+  <xacro:property name="base_length" value="0.2667"/>  <!-- 266.7mm -->
+  <xacro:property name="base_width" value="0.102"/>   <!-- 102mm main body width -->
+  <xacro:property name="base_height" value="0.090"/>  <!-- 90mm -->
+  <xacro:property name="track_width" value="0.042"/>   <!-- 42mm tread width -->
+  <xacro:property name="track_length" value="0.2667"/> <!-- Same as body length -->
+  <xacro:property name="track_height" value="0.090"/>  <!-- Same as body height -->
+  <xacro:property name="wheel_radius" value="0.045"/>  <!-- Half of track height -->
+  <xacro:property name="wheel_separation" value="0.144"/> <!-- 102mm + 42mm = center to center -->
   <!-- Materials -->
   <material name="red">
@@ -26,4 +30,8 @@
     <color rgba="1.0 1.0 1.0 1.0"/>
   </material>
+  <!-- Root Link (dummy link to fix KDL warning) -->
+  <link name="base_footprint">
+    <!-- No inertia, visual, or collision for dummy link -->
+  </link>
   <!-- Base Link (main chassis) -->
   <link name="base_link">
@@ -43,66 +51,66 @@
     <inertial>
       <origin xyz="0 0 0" rpy="0 0 0"/>
-      <mass value="50.0"/>
-      <inertia ixx="4.17" ixy="0.0" ixz="0.0" iyy="2.5" iyz="0.0" izz="4.17"/>
+      <mass value="5.0"/>
+      <inertia ixx="0.08" ixy="0.0" ixz="0.0" iyy="0.15" iyz="0.0" izz="0.18"/>
     </inertial>
   </link>
   <!-- Left Track -->
   <link name="left_wheel">
-    <!-- Main track body (wider cylinder) -->
-    <visual>
-      <origin xyz="0 0 0" rpy="${PI/2} 0 0"/>
-      <geometry>
-        <cylinder radius="${wheel_radius}" length="${wheel_width}"/>
-      </geometry>
-      <material name="black"/>
-    </visual>
-    <!-- Track tread bottom (fixed to wheel origin) -->
-    <visual>
-      <origin xyz="0 0 ${-wheel_radius + 0.01}" rpy="0 0 0"/>
-      <geometry>
-        <box size="${track_length} ${wheel_width * 0.9} 0.02"/>
-      </geometry>
-      <material name="black"/>
-    </visual>
-    <collision>
-      <origin xyz="0 0 0" rpy="${PI/2} 0 0"/>
-      <geometry>
-        <cylinder radius="${wheel_radius}" length="${wheel_width}"/>
-      </geometry>
-    </collision>
-    <inertial>
-      <origin xyz="0 0 0" rpy="${PI/2} 0 0"/>
-      <mass value="5.0"/>
-      <inertia ixx="0.06" ixy="0.0" ixz="0.0" iyy="0.06" iyz="0.0" izz="0.11"/>
+    <!-- Main track body (rectangular track shape) -->
+    <visual>
+      <origin xyz="0 0 0" rpy="0 0 0"/>
+      <geometry>
+        <box size="${track_length} ${track_width} ${track_height}"/>
+      </geometry>
+      <material name="black"/>
+    </visual>
+    <!-- Track tread pattern -->
+    <visual>
+      <origin xyz="0 0 ${-track_height/2 + 0.005}" rpy="0 0 0"/>
+      <geometry>
+        <box size="${track_length * 0.9} ${track_width * 0.8} 0.01"/>
+      </geometry>
+      <material name="black"/>
+    </visual>
+    <collision>
+      <origin xyz="0 0 0" rpy="0 0 0"/>
+      <geometry>
+        <box size="${track_length} ${track_width} ${track_height}"/>
+      </geometry>
+    </collision>
+    <inertial>
+      <origin xyz="0 0 0" rpy="0 0 0"/>
+      <mass value="2.0"/>
+      <inertia ixx="0.02" ixy="0.0" ixz="0.0" iyy="0.02" iyz="0.0" izz="0.03"/>
     </inertial>
   </link>
   <!-- Right Track -->
   <link name="right_wheel">
-    <!-- Main track body (wider cylinder) -->
-    <visual>
-      <origin xyz="0 0 0" rpy="${PI/2} 0 0"/>
-      <geometry>
-        <cylinder radius="${wheel_radius}" length="${wheel_width}"/>
-      </geometry>
-      <material name="black"/>
-    </visual>
-    <!-- Track tread bottom (fixed to wheel origin) -->
-    <visual>
-      <origin xyz="0 0 ${-wheel_radius + 0.01}" rpy="0 0 0"/>
-      <geometry>
-        <box size="${track_length} ${wheel_width * 0.9} 0.02"/>
-      </geometry>
-      <material name="black"/>
-    </visual>
-    <collision>
-      <origin xyz="0 0 0" rpy="${PI/2} 0 0"/>
-      <geometry>
-        <cylinder radius="${wheel_radius}" length="${wheel_width}"/>
-      </geometry>
-    </collision>
-    <inertial>
-      <origin xyz="0 0 0" rpy="${PI/2} 0 0"/>
-      <mass value="5.0"/>
-      <inertia ixx="0.06" ixy="0.0" ixz="0.0" iyy="0.06" iyz="0.0" izz="0.11"/>
+    <!-- Main track body (rectangular track shape) -->
+    <visual>
+      <origin xyz="0 0 0" rpy="0 0 0"/>
+      <geometry>
+        <box size="${track_length} ${track_width} ${track_height}"/>
+      </geometry>
+      <material name="black"/>
+    </visual>
+    <!-- Track tread pattern -->
+    <visual>
+      <origin xyz="0 0 ${-track_height/2 + 0.005}" rpy="0 0 0"/>
+      <geometry>
+        <box size="${track_length * 0.9} ${track_width * 0.8} 0.01"/>
+      </geometry>
+      <material name="black"/>
+    </visual>
+    <collision>
+      <origin xyz="0 0 0" rpy="0 0 0"/>
+      <geometry>
+        <box size="${track_length} ${track_width} ${track_height}"/>
+      </geometry>
+    </collision>
+    <inertial>
+      <origin xyz="0 0 0" rpy="0 0 0"/>
+      <mass value="2.0"/>
+      <inertia ixx="0.02" ixy="0.0" ixz="0.0" iyy="0.02" iyz="0.0" izz="0.03"/>
     </inertial>
   </link>
@@ -128,10 +136,19 @@
     </inertial>
   </link>
-  <!-- GPS Link -->
+  <!-- HGLRC M100-5883 GPS Module (M10 chip, 21x21x8.02mm, 7.73g) -->
   <link name="gps_link">
-    <visual>
-      <origin xyz="0 0 0" rpy="0 0 0"/>
-      <geometry>
-        <box size="0.05 0.05 0.02"/>
+    <!-- Main PCB board -->
+    <visual>
+      <origin xyz="0 0 0" rpy="0 0 0"/>
+      <geometry>
+        <box size="0.021 0.021 0.008"/>  <!-- 21x21x8mm actual size -->
+      </geometry>
+      <material name="blue"/>
+    </visual>
+    <!-- Ceramic antenna (integrated on PCB) -->
+    <visual>
+      <origin xyz="0 0 0.004" rpy="0 0 0"/>
+      <geometry>
+        <box size="0.015 0.015 0.002"/>  <!-- 15x15x2mm ceramic patch -->
       </geometry>
       <material name="white"/>
@@ -140,32 +157,33 @@
       <origin xyz="0 0 0" rpy="0 0 0"/>
       <geometry>
-        <box size="0.05 0.05 0.02"/>
-      </geometry>
-    </collision>
-    <inertial>
-      <origin xyz="0 0 0" rpy="0 0 0"/>
-      <mass value="0.05"/>
-      <inertia ixx="0.0001" ixy="0.0" ixz="0.0" iyy="0.0001" iyz="0.0" izz="0.0001"/>
-    </inertial>
-  </link>
-  <!-- Compass Link -->
+        <box size="0.021 0.021 0.008"/>  <!-- Actual dimensions -->
+      </geometry>
+    </collision>
+    <inertial>
+      <origin xyz="0 0 0" rpy="0 0 0"/>
+      <mass value="0.00773"/>  <!-- 7.73g actual weight -->
+      <inertia ixx="0.000003" ixy="0.0" ixz="0.0" iyy="0.000003" iyz="0.0" izz="0.000005"/>
+    </inertial>
+  </link>
+  <!-- QMC5883 Compass/Magnetometer (integrated in GPS module) -->
   <link name="compass_link">
-    <visual>
-      <origin xyz="0 0 0" rpy="0 0 0"/>
-      <geometry>
-        <cylinder radius="0.02" length="0.01"/>
-      </geometry>
-      <material name="red"/>
-    </visual>
-    <collision>
-      <origin xyz="0 0 0" rpy="0 0 0"/>
-      <geometry>
-        <cylinder radius="0.02" length="0.01"/>
-      </geometry>
-    </collision>
-    <inertial>
-      <origin xyz="0 0 0" rpy="0 0 0"/>
-      <mass value="0.02"/>
-      <inertia ixx="0.00001" ixy="0.0" ixz="0.0" iyy="0.00001" iyz="0.0" izz="0.00001"/>
+    <!-- Small magnetometer chip representation -->
+    <visual>
+      <origin xyz="0 0 0" rpy="0 0 0"/>
+      <geometry>
+        <box size="0.003 0.003 0.001"/>  <!-- 3x3x1mm chip size -->
+      </geometry>
+      <material name="black"/>
+    </visual>
+    <collision>
+      <origin xyz="0 0 0" rpy="0 0 0"/>
+      <geometry>
+        <box size="0.003 0.003 0.001"/>
+      </geometry>
+    </collision>
+    <inertial>
+      <origin xyz="0 0 0" rpy="0 0 0"/>
+      <mass value="0.001"/>  <!-- Negligible mass -->
+      <inertia ixx="0.000001" ixy="0.0" ixz="0.0" iyy="0.000001" iyz="0.0" izz="0.000001"/>
     </inertial>
   </link>
@@ -214,17 +232,23 @@
   <!-- Sprayer tank removed -->
   <!-- Joints -->
-  <!-- Left Wheel Joint -->
+  <!-- Base Footprint to Base Link Joint -->
+  <joint name="base_footprint_joint" type="fixed">
+    <parent link="base_footprint"/>
+    <child link="base_link"/>
+    <origin xyz="0 0 ${base_height/2}" rpy="0 0 0"/>
+  </joint>
+  <!-- Left Track Joint -->
   <joint name="left_wheel_joint" type="continuous">
     <parent link="base_link"/>
     <child link="left_wheel"/>
-    <origin xyz="0 ${wheel_separation/2} ${-base_height/2 + wheel_radius}" rpy="0 0 0"/>
+    <origin xyz="0 ${(base_width + track_width)/2} 0" rpy="0 0 0"/>
     <axis xyz="0 1 0"/>
     <dynamics damping="1.0" friction="0.1"/>
   </joint>
-  <!-- Right Wheel Joint -->
+  <!-- Right Track Joint -->
   <joint name="right_wheel_joint" type="continuous">
     <parent link="base_link"/>
     <child link="right_wheel"/>
-    <origin xyz="0 ${-wheel_separation/2} ${-base_height/2 + wheel_radius}" rpy="0 0 0"/>
+    <origin xyz="0 ${-(base_width + track_width)/2} 0" rpy="0 0 0"/>
     <axis xyz="0 1 0"/>
     <dynamics damping="1.0" friction="0.1"/>
@@ -242,9 +266,9 @@
     <origin xyz="0 0 ${base_height/2 + 0.15}" rpy="0 0 0"/>
   </joint>
-  <!-- Compass Joint -->
+  <!-- Compass Joint (QMC5883 integrated on GPS PCB) -->
   <joint name="compass_joint" type="fixed">
     <parent link="gps_link"/>
     <child link="compass_link"/>
-    <origin xyz="0 0 0.03" rpy="0 0 0"/>
+    <origin xyz="0.008 0.008 0.002" rpy="0 0 0"/>  <!-- Positioned on 21x21mm GPS PCB -->
   </joint>
   <!-- Mower Deck Joint -->
@@ -290,5 +314,5 @@
   </gazebo>
   <gazebo reference="compass_link">
-    <material>Gazebo/Red</material>
+    <material>Gazebo/Black</material>
   </gazebo>
   <gazebo reference="mower_deck">
@@ -348,5 +372,5 @@
       <publish_wheel_tf>true</publish_wheel_tf>
       <odometry_frame>odom</odometry_frame>
-      <robot_base_frame>base_link</robot_base_frame>
+      <robot_base_frame>base_footprint</robot_base_frame>
     </plugin>
   </gazebo>
@@ -413,16 +437,101 @@
     </sensor>
   </gazebo>
-  <!-- GPS Plugin -->
+  <!-- HGLRC M100-5883 GPS Plugin (M10 chip, multi-constellation) -->
   <gazebo reference="gps_link">
-    <sensor type="gps" name="gps_sensor">
-      <update_rate>10.0</update_rate>
+    <sensor type="gps" name="hglrc_m100_gps">
+      <update_rate>10.0</update_rate>  <!-- 10Hz output frequency -->
       <plugin name="gps_controller" filename="libgazebo_ros_gps_sensor.so">
         <ros>
-          <namespace>gps</namespace>
+          <namespace>hglrc_gps</namespace>
           <remapping>fix:=fix</remapping>
+          <remapping>vel:=vel</remapping>
         </ros>
         <frame_name>gps_link</frame_name>
+        <!-- M10 chip specifications -->
+        <position_sensing>
+          <horizontal>
+            <noise type="gaussian">
+              <mean>0.0</mean>
+              <stddev>2.5</stddev>  <!-- ~2.5m CEP typical for consumer GPS -->
+            </noise>
+          </horizontal>
+          <vertical>
+            <noise type="gaussian">
+              <mean>0.0</mean>
+              <stddev>4.0</stddev>  <!-- Vertical accuracy typically worse -->
+            </noise>
+          </vertical>
+        </position_sensing>
+        <velocity_sensing>
+          <horizontal>
+            <noise type="gaussian">
+              <mean>0.0</mean>
+              <stddev>0.1</stddev>
+            </noise>
+          </horizontal>
+          <vertical>
+            <noise type="gaussian">
+              <mean>0.0</mean>
+              <stddev>0.1</stddev>
+            </noise>
+          </vertical>
+        </velocity_sensing>
       </plugin>
     </sensor>
   </gazebo>
+  <!-- QMC5883 Magnetometer Plugin -->
+  <gazebo reference="compass_link">
+    <sensor type="magnetometer" name="qmc5883_compass">
+      <update_rate>100.0</update_rate>  <!-- High update rate for compass -->
+      <plugin name="magnetometer_controller" filename="libgazebo_ros_imu_sensor.so">
+        <ros>
+          <namespace>hglrc_gps</namespace>
+          <remapping>imu:=compass</remapping>
+        </ros>
+        <frame_name>compass_link</frame_name>
+        <initial_orientation_as_reference>false</initial_orientation_as_reference>
+        <!-- QMC5883 specifications -->
+        <angular_velocity>
+          <x>
+            <noise type="gaussian">
+              <mean>0.0</mean>
+              <stddev>0.0</stddev>
+            </noise>
+          </x>
+          <y>
+            <noise type="gaussian">
+              <mean>0.0</mean>
+              <stddev>0.0</stddev>
+            </noise>
+          </y>
+          <z>
+            <noise type="gaussian">
+              <mean>0.0</mean>
+              <stddev>0.0</stddev>
+            </noise>
+          </z>
+        </angular_velocity>
+        <linear_acceleration>
+          <x>
+            <noise type="gaussian">
+              <mean>0.0</mean>
+              <stddev>0.0</stddev>
+            </noise>
+          </x>
+          <y>
+            <noise type="gaussian">
+              <mean>0.0</mean>
+              <stddev>0.0</stddev>
+            </noise>
+          </y>
+          <z>
+            <noise type="gaussian">
+              <mean>0.0</mean>
+              <stddev>0.0</stddev>
+            </noise>
+          </z>
+        </linear_acceleration>
+      </plugin>
+    </sensor>
+  </gazebo>
 </robot>

Commit message: checkpoint2

File: install/tractor_bringup/share/tractor_bringup/urdf/tractor.urdf.xacro (robot description, xacro)
@@ -8,5 +8,5 @@
   <xacro:property name="base_length" value="0.2667"/>  <!-- 266.7mm -->
   <xacro:property name="base_width" value="0.102"/>   <!-- 102mm main body width -->
-  <xacro:property name="base_height" value="0.090"/>  <!-- 90mm -->
+  <xacro:property name="base_height" value="0.058"/>  <!-- 58mm -->
   <xacro:property name="track_width" value="0.042"/>   <!-- 42mm tread width -->
   <xacro:property name="track_length" value="0.2667"/> <!-- Same as body length -->
@@ -189,4 +189,5 @@
   </link>
   <!-- Mower Deck Link -->
+  <!--
   <link name="mower_deck">
     <visual>
@@ -209,4 +210,5 @@
     </inertial>
   </link>
+  -->
   <!-- Laser Scanner Link -->
   <link name="laser">
@@ -242,5 +244,5 @@
     <parent link="base_link"/>
     <child link="left_wheel"/>
-    <origin xyz="0 ${(base_width + track_width)/2} 0" rpy="0 0 0"/>
+    <origin xyz="0 ${(base_width + track_width)/2} -0.016" rpy="0 0 0"/>
     <axis xyz="0 1 0"/>
     <dynamics damping="1.0" friction="0.1"/>
@@ -250,5 +252,5 @@
     <parent link="base_link"/>
     <child link="right_wheel"/>
-    <origin xyz="0 ${-(base_width + track_width)/2} 0" rpy="0 0 0"/>
+    <origin xyz="0 ${-(base_width + track_width)/2} -0.016" rpy="0 0 0"/>
     <axis xyz="0 1 0"/>
     <dynamics damping="1.0" friction="0.1"/>
@@ -273,4 +275,5 @@
   </joint>
   <!-- Mower Deck Joint -->
+  <!--
   <joint name="mower_deck_joint" type="fixed">
     <parent link="base_link"/>
@@ -278,4 +281,5 @@
     <origin xyz="${base_length/2 + 0.3} 0 ${-base_height/2 - 0.05}" rpy="0 0 0"/>
   </joint>
+  -->
   <!-- Laser Joint -->
   <joint name="laser_joint" type="fixed">
@@ -316,7 +320,9 @@
     <material>Gazebo/Black</material>
   </gazebo>
+  <!--
   <gazebo reference="mower_deck">
     <material>Gazebo/Red</material>
   </gazebo>
+  -->
   <gazebo reference="laser">
     <material>Gazebo/Black</material>
