Commit message: Update tractor URDF: remove radar, add platform, relocate camera

File: src/tractor_bringup/urdf/tractor.urdf.xacro (robot description, xacro)
@@ -14,4 +14,7 @@
   <xacro:property name="wheel_radius" value="0.045"/>  <!-- Half of track height -->
   <xacro:property name="wheel_separation" value="0.144"/> <!-- 102mm + 42mm = center to center -->
+  <!-- Platform properties -->
+  <xacro:property name="platform_height" value="0.0025"/> <!-- 2.5mm -->
+  <xacro:property name="platform_offset_z" value="0.05"/>  <!-- 50mm -->
   <!-- Materials -->
   <material name="red">
@@ -120,5 +123,5 @@
       <origin xyz="0 0 0" rpy="0 0 0"/>
       <geometry>
-        <box size="0.09 0.025 0.025"/>
+        <box size="0.09 0.025 0.025"/> <!-- Updated dimensions -->
       </geometry>
       <material name="black"/>
@@ -127,10 +130,10 @@
       <origin xyz="0 0 0" rpy="0 0 0"/>
       <geometry>
-        <box size="0.09 0.025 0.025"/>
-      </geometry>
-    </collision>
-    <inertial>
-      <origin xyz="0 0 0" rpy="0 0 0"/>
-      <mass value="0.1"/>
+        <box size="0.09 0.025 0.025"/> <!-- Updated dimensions -->
+      </geometry>
+    </collision>
+    <inertial>
+      <origin xyz="0 0 0" rpy="0 0 0"/>
+      <mass value="0.1"/> <!-- Mass can be re-evaluated if needed -->
       <inertia ixx="0.001" ixy="0.0" ixz="0.0" iyy="0.001" iyz="0.0" izz="0.001"/>
     </inertial>
@@ -211,26 +214,27 @@
   </link>
   -->
-  <!-- Laser Scanner Link -->
-  <link name="laser">
-    <visual>
-      <origin xyz="0 0 0" rpy="0 0 0"/>
-      <geometry>
-        <cylinder radius="0.05" length="0.07"/>
-      </geometry>
-      <material name="black"/>
-    </visual>
-    <collision>
-      <origin xyz="0 0 0" rpy="0 0 0"/>
-      <geometry>
-        <cylinder radius="0.05" length="0.07"/>
-      </geometry>
-    </collision>
-    <inertial>
-      <origin xyz="0 0 0" rpy="0 0 0"/>
-      <mass value="0.3"/>
-      <inertia ixx="0.001" ixy="0.0" ixz="0.0" iyy="0.001" iyz="0.0" izz="0.001"/>
-    </inertial>
-  </link>
+  <!-- Laser Scanner Link REMOVED -->
   <!-- Sprayer tank removed -->
+  <!-- Platform Link -->
+  <link name="platform_link">
+    <visual>
+      <origin xyz="0 0 0" rpy="0 0 0"/>
+      <geometry>
+        <box size="${base_length} ${base_width} ${platform_height}"/>
+      </geometry>
+      <material name="blue"/>
+    </visual>
+    <collision>
+      <origin xyz="0 0 0" rpy="0 0 0"/>
+      <geometry>
+        <box size="${base_length} ${base_width} ${platform_height}"/>
+      </geometry>
+    </collision>
+    <inertial>
+      <origin xyz="0 0 0" rpy="0 0 0"/>
+      <mass value="0.5"/> <!-- Estimated mass -->
+      <inertia ixx="0.001" ixy="0.0" ixz="0.0" iyy="0.001" iyz="0.0" izz="0.001"/> <!-- Estimated inertia -->
+    </inertial>
+  </link>
   <!-- Joints -->
   <!-- Base Footprint to Base Link Joint -->
@@ -254,20 +258,10 @@
   <!-- Camera Joint -->
   <joint name="camera_joint" type="fixed">
-    <parent link="base_link"/>
+    <parent link="platform_link"/> <!-- Changed parent to platform_link -->
     <child link="camera_link"/>
-    <origin xyz="${base_length/2 - 0.05} 0 ${base_height/2 + 0.1}" rpy="0 0 0"/>
-  </joint>
-  <!-- GPS Joint -->
-  <joint name="gps_joint" type="fixed">
-    <parent link="base_link"/>
-    <child link="gps_link"/>
-    <origin xyz="0 0 ${base_height/2 + 0.15}" rpy="0 0 0"/>
-  </joint>
-  <!-- Compass Joint (QMC5883 integrated on GPS PCB) -->
-  <joint name="compass_joint" type="fixed">
-    <parent link="gps_link"/>
-    <child link="compass_link"/>
-    <origin xyz="0.008 0.008 0.002" rpy="0 0 0"/>  <!-- Positioned on 21x21mm GPS PCB -->
-  </joint>
+    <origin xyz="${base_length/2 - 0.09/2} 0 ${platform_height/2 + 0.025/2}" rpy="0 0 0"/> <!-- Adjusted origin -->
+  </joint>
+  <!-- GPS Joint REMOVED -->
+  <!-- Compass Joint REMOVED -->
   <!-- Mower Deck Joint -->
   <!--
@@ -278,11 +272,12 @@
   </joint>
   -->
-  <!-- Laser Joint -->
-  <joint name="laser_joint" type="fixed">
+  <!-- Laser Joint REMOVED -->
+  <!-- Sprayer tank joint removed -->
+  <!-- Platform Joint -->
+  <joint name="platform_joint" type="fixed">
     <parent link="base_link"/>
-    <child link="laser"/>
-    <origin xyz="${base_length/2 - 0.1} 0 ${base_height/2 + 0.05}" rpy="0 0 0"/>
-  </joint>
-  <!-- Sprayer tank joint removed -->
+    <child link="platform_link"/>
+    <origin xyz="0 0 ${base_height/2 + platform_offset_z + platform_height/2}" rpy="0 0 0"/>
+  </joint>
   <!-- Virtual Visualization Wheels (small, for motion display only) -->
   <!-- These rotate to show movement while tank tracks stay fixed -->
@@ -342,13 +337,16 @@
     <maxVel>1.0</maxVel>
   </gazebo>
+  <gazebo reference="platform_link">
+    <material>Gazebo/Blue</material>
+  </gazebo>
   <gazebo reference="camera_link">
     <material>Gazebo/Black</material>
   </gazebo>
-  <gazebo reference="gps_link">
-    <material>Gazebo/White</material>
-  </gazebo>
-  <gazebo reference="compass_link">
-    <material>Gazebo/Black</material>
-  </gazebo>
+  <!-- <gazebo reference="gps_link"> -->
+    <!-- <material>Gazebo/White</material> -->
+  <!-- </gazebo> -->
+  <!-- <gazebo reference="compass_link"> -->
+    <!-- <material>Gazebo/Black</material> -->
+  <!-- </gazebo> -->
   <!--
   <gazebo reference="mower_deck">
@@ -356,37 +354,37 @@
   </gazebo>
   -->
-  <gazebo reference="laser">
-    <material>Gazebo/Black</material>
-    <sensor type="ray" name="laser_scanner">
-      <update_rate>40</update_rate>
-      <ray>
-        <scan>
-          <horizontal>
-            <samples>720</samples>
-            <resolution>1</resolution>
-            <min_angle>0.0</min_angle>
-            <max_angle>6.28318530718</max_angle>
-          </horizontal>
-        </scan>
-        <range>
-          <min>0.1</min>
-          <max>10.0</max>
-          <resolution>0.01</resolution>
-        </range>
-        <noise>
-          <type>gaussian</type>
-          <mean>0.0</mean>
-          <stddev>0.01</stddev>
-        </noise>
-      </ray>
-      <plugin name="gazebo_ros_laser" filename="libgazebo_ros_ray_sensor.so">
-        <ros>
-          <remapping>~/out:=scan</remapping>
-        </ros>
-        <output_type>sensor_msgs/LaserScan</output_type>
-        <frame_name>laser</frame_name>
-      </plugin>
-    </sensor>
-  </gazebo>
+  <!-- <gazebo reference="laser"> -->
+    <!-- <material>Gazebo/Black</material> -->
+    <!-- <sensor type="ray" name="laser_scanner"> -->
+      <!-- <update_rate>40</update_rate> -->
+      <!-- <ray> -->
+        <!-- <scan> -->
+          <!-- <horizontal> -->
+            <!-- <samples>720</samples> -->
+            <!-- <resolution>1</resolution> -->
+            <!-- <min_angle>0.0</min_angle> -->
+            <!-- <max_angle>6.28318530718</max_angle> -->
+          <!-- </horizontal> -->
+        <!-- </scan> -->
+        <!-- <range> -->
+          <!-- <min>0.1</min> -->
+          <!-- <max>10.0</max> -->
+          <!-- <resolution>0.01</resolution> -->
+        <!-- </range> -->
+        <!-- <noise> -->
+          <!-- <type>gaussian</type> -->
+          <!-- <mean>0.0</mean> -->
+          <!-- <stddev>0.01</stddev> -->
+        <!-- </noise> -->
+      <!-- </ray> -->
+      <!-- <plugin name="gazebo_ros_laser" filename="libgazebo_ros_ray_sensor.so"> -->
+        <!-- <ros> -->
+          <!-- <remapping>~/out:=scan</remapping> -->
+        <!-- </ros> -->
+        <!-- <output_type>sensor_msgs/LaserScan</output_type> -->
+        <!-- <frame_name>laser</frame_name> -->
+      <!-- </plugin> -->
+    <!-- </sensor> -->
+  <!-- </gazebo> -->
   <!-- Sprayer tank Gazebo reference removed -->
   <!-- Differential Drive Plugin - Disabled for fixed track joints -->
@@ -477,101 +475,99 @@
     </sensor>
   </gazebo>
-  <!-- HGLRC M100-5883 GPS Plugin (M10 chip, multi-constellation) -->
-  <gazebo reference="gps_link">
-    <sensor type="gps" name="hglrc_m100_gps">
-      <update_rate>10.0</update_rate>  <!-- 10Hz output frequency -->
-      <plugin name="gps_controller" filename="libgazebo_ros_gps_sensor.so">
-        <ros>
-          <namespace>hglrc_gps</namespace>
-          <remapping>fix:=fix</remapping>
-          <remapping>vel:=vel</remapping>
-        </ros>
-        <frame_name>gps_link</frame_name>
-        <!-- M10 chip specifications -->
-        <position_sensing>
-          <horizontal>
-            <noise type="gaussian">
-              <mean>0.0</mean>
-              <stddev>2.5</stddev>  <!-- ~2.5m CEP typical for consumer GPS -->
-            </noise>
-          </horizontal>
-          <vertical>
-            <noise type="gaussian">
-              <mean>0.0</mean>
-              <stddev>4.0</stddev>  <!-- Vertical accuracy typically worse -->
-            </noise>
-          </vertical>
-        </position_sensing>
-        <velocity_sensing>
-          <horizontal>
-            <noise type="gaussian">
-              <mean>0.0</mean>
-              <stddev>0.1</stddev>
-            </noise>
-          </horizontal>
-          <vertical>
-            <noise type="gaussian">
-              <mean>0.0</mean>
-              <stddev>0.1</stddev>
-            </noise>
-          </vertical>
-        </velocity_sensing>
-      </plugin>
-    </sensor>
-  </gazebo>
-  <!-- QMC5883 Magnetometer Plugin -->
-  <gazebo reference="compass_link">
-    <sensor type="magnetometer" name="qmc5883_compass">
-      <update_rate>100.0</update_rate>  <!-- High update rate for compass -->
-      <plugin name="magnetometer_controller" filename="libgazebo_ros_imu_sensor.so">
-        <ros>
-          <namespace>hglrc_gps</namespace>
-          <remapping>imu:=compass</remapping>
-        </ros>
-        <frame_name>compass_link</frame_name>
-        <initial_orientation_as_reference>false</initial_orientation_as_reference>
-        <!-- QMC5883 specifications -->
-        <angular_velocity>
-          <x>
-            <noise type="gaussian">
-              <mean>0.0</mean>
-              <stddev>0.0</stddev>
-            </noise>
-          </x>
-          <y>
-            <noise type="gaussian">
-              <mean>0.0</mean>
-              <stddev>0.0</stddev>
-            </noise>
-          </y>
-          <z>
-            <noise type="gaussian">
-              <mean>0.0</mean>
-              <stddev>0.0</stddev>
-            </noise>
-          </z>
-        </angular_velocity>
-        <linear_acceleration>
-          <x>
-            <noise type="gaussian">
-              <mean>0.0</mean>
-              <stddev>0.0</stddev>
-            </noise>
-          </x>
-          <y>
-            <noise type="gaussian">
-              <mean>0.0</mean>
-              <stddev>0.0</stddev>
-            </noise>
-          </y>
-          <z>
-            <noise type="gaussian">
-              <mean>0.0</mean>
-              <stddev>0.0</stddev>
-            </noise>
-          </z>
-        </linear_acceleration>
-      </plugin>
-    </sensor>
-  </gazebo>
+  <!-- HGLRC M100-5883 GPS Plugin (M10 chip, multi-constellation) REMOVED -->
+  <!-- <gazebo reference="gps_link"> -->
+    <!-- <sensor type="gps" name="hglrc_m100_gps"> -->
+      <!-- <update_rate>10.0</update_rate>  -->
+      <!-- <plugin name="gps_controller" filename="libgazebo_ros_gps_sensor.so"> -->
+        <!-- <ros> -->
+          <!-- <namespace>hglrc_gps</namespace> -->
+          <!-- <remapping>fix:=fix</remapping> -->
+          <!-- <remapping>vel:=vel</remapping> -->
+        <!-- </ros> -->
+        <!-- <frame_name>gps_link</frame_name> -->
+        <!-- <position_sensing> -->
+          <!-- <horizontal> -->
+            <!-- <noise type="gaussian"> -->
+              <!-- <mean>0.0</mean> -->
+              <!-- <stddev>2.5</stddev>   -->
+            <!-- </noise> -->
+          <!-- </horizontal> -->
+          <!-- <vertical> -->
+            <!-- <noise type="gaussian"> -->
+              <!-- <mean>0.0</mean> -->
+              <!-- <stddev>4.0</stddev>   -->
+            <!-- </noise> -->
+          <!-- </vertical> -->
+        <!-- </position_sensing> -->
+        <!-- <velocity_sensing> -->
+          <!-- <horizontal> -->
+            <!-- <noise type="gaussian"> -->
+              <!-- <mean>0.0</mean> -->
+              <!-- <stddev>0.1</stddev> -->
+            <!-- </noise> -->
+          <!-- </horizontal> -->
+          <!-- <vertical> -->
+            <!-- <noise type="gaussian"> -->
+              <!-- <mean>0.0</mean> -->
+              <!-- <stddev>0.1</stddev> -->
+            <!-- </noise> -->
+          <!-- </vertical> -->
+        <!-- </velocity_sensing> -->
+      <!-- </plugin> -->
+    <!-- </sensor> -->
+  <!-- </gazebo> -->
+  <!-- QMC5883 Magnetometer Plugin REMOVED -->
+  <!-- <gazebo reference="compass_link"> -->
+    <!-- <sensor type="magnetometer" name="qmc5883_compass"> -->
+      <!-- <update_rate>100.0</update_rate>   -->
+      <!-- <plugin name="magnetometer_controller" filename="libgazebo_ros_imu_sensor.so"> -->
+        <!-- <ros> -->
+          <!-- <namespace>hglrc_gps</namespace> -->
+          <!-- <remapping>imu:=compass</remapping> -->
+        <!-- </ros> -->
+        <!-- <frame_name>compass_link</frame_name> -->
+        <!-- <initial_orientation_as_reference>false</initial_orientation_as_reference> -->
+        <!-- <angular_velocity> -->
+          <!-- <x> -->
+            <!-- <noise type="gaussian"> -->
+              <!-- <mean>0.0</mean> -->
+              <!-- <stddev>0.0</stddev> -->
+            <!-- </noise> -->
+          <!-- </x> -->
+          <!-- <y> -->
+            <!-- <noise type="gaussian"> -->
+              <!-- <mean>0.0</mean> -->
+              <!-- <stddev>0.0</stddev> -->
+            <!-- </noise> -->
+          <!-- </y> -->
+          <!-- <z> -->
+            <!-- <noise type="gaussian"> -->
+              <!-- <mean>0.0</mean> -->
+              <!-- <stddev>0.0</stddev> -->
+            <!-- </noise> -->
+          <!-- </z> -->
+        <!-- </angular_velocity> -->
+        <!-- <linear_acceleration> -->
+          <!-- <x> -->
+            <!-- <noise type="gaussian"> -->
+              <!-- <mean>0.0</mean> -->
+              <!-- <stddev>0.0</stddev> -->
+            <!-- </noise> -->
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