Commit message: fix: Correct camera and LiDAR positions in URDF and update camera height parameter in occupancy grid processing.

File: src/tractor_bringup/urdf/tractor.urdf.xacro (robot description, xacro)
@@ -264,10 +264,10 @@
       <origin xyz="0 0 0" rpy="0 0 0"/>
       <geometry>
-        <cylinder radius="0.019" length="0.041"/>
+        <cylinder radius="0.019" length="0.035"/>
       </geometry>
       <material name="black"/>
     </visual>
     <visual>
-      <origin xyz="0 0 0.025" rpy="0 0 0"/>
+      <origin xyz="0 0 0.0175" rpy="0 0 0"/>
       <geometry>
         <cylinder radius="0.015" length="0.008"/>
@@ -278,5 +278,5 @@
       <origin xyz="0 0 0" rpy="0 0 0"/>
       <geometry>
-        <cylinder radius="0.019" length="0.041"/>
+        <cylinder radius="0.019" length="0.035"/>
       </geometry>
     </collision>
@@ -312,5 +312,7 @@
     <!-- Camera: 25mm deep, front flush with platform edge at base_length/2 (133.35mm) -->
     <!-- Camera center at: 133.35 - 12.5 = 120.85mm = 0.12085m from base_link center -->
-    <origin xyz="0.12085 0 ${platform_height/2 + 0.025/2}" rpy="0 0 0"/>
+    <!-- Measured camera bottom: 174mm from ground, optical center at 186.5mm -->
+    <!-- Platform at 109.25mm, so offset = 186.5 - 109.25 = 77.25mm -->
+    <origin xyz="0.12085 0 0.07725" rpy="0 0 0"/>
   </joint>
   <!-- GPS Joint REMOVED -->
@@ -344,7 +346,8 @@
     <!-- LiDAR: 38mm diameter, front is 38mm behind camera front -->
     <!-- Camera front at 133.35mm, LiDAR front at 95.35mm, LiDAR center at 76.35mm = 0.07635m -->
-    <!-- Z: 200mm from ground = 171mm above base_link + 20.5mm to center = 191.5mm = 0.1915m -->
+    <!-- Measured: Camera top (199mm) + 3mm gap + 35mm/2 = 219.5mm from ground -->
+    <!-- base_link at 29mm, so offset = 219.5 - 29 = 190.5mm = 0.1905m -->
     <!-- Arrow points forward, no rotation needed - counterclockwise scan for correct orientation -->
-    <origin xyz="0.07635 0 0.1915" rpy="0 0 0"/>
+    <origin xyz="0.07635 0 0.1905" rpy="0 0 0"/>
   </joint>
   <!-- Virtual Visualization Wheels (small, for motion display only) -->

Commit message: camera height

File: src/tractor_bringup/urdf/tractor.urdf.xacro (robot description, xacro)
@@ -312,7 +312,7 @@
     <!-- Camera: 25mm deep, front flush with platform edge at base_length/2 (133.35mm) -->
     <!-- Camera center at: 133.35 - 12.5 = 120.85mm = 0.12085m from base_link center -->
-    <!-- Measured camera bottom: 174mm from ground, optical center at 186.5mm -->
-    <!-- Platform at 109.25mm, so offset = 186.5 - 109.25 = 77.25mm -->
-    <origin xyz="0.12085 0 0.07725" rpy="0 0 0"/>
+    <!-- Camera mount tower raised 175mm: optical center now 186.5 + 175 = 361.5mm from ground -->
+    <!-- Platform at 109.25mm, so offset = 361.5 - 109.25 = 252.25mm -->
+    <origin xyz="0.12085 0 0.25225" rpy="0 0 0"/>
   </joint>
   <!-- GPS Joint REMOVED -->
@@ -347,7 +347,8 @@
     <!-- Camera front at 133.35mm, LiDAR front at 95.35mm, LiDAR center at 76.35mm = 0.07635m -->
     <!-- Measured: Camera top (199mm) + 3mm gap + 35mm/2 = 219.5mm from ground -->
-    <!-- base_link at 29mm, so offset = 219.5 - 29 = 190.5mm = 0.1905m -->
+    <!-- Camera mount tower raised 175mm, LiDAR rides with it: 219.5 + 175 = 394.5mm from ground -->
+    <!-- base_link at 29mm, so offset = 394.5 - 29 = 365.5mm = 0.3655m -->
     <!-- Arrow points forward, no rotation needed - counterclockwise scan for correct orientation -->
-    <origin xyz="0.07635 0 0.1905" rpy="0 0 0"/>
+    <origin xyz="0.07635 0 0.3655" rpy="0 0 0"/>
   </joint>
   <!-- Virtual Visualization Wheels (small, for motion display only) -->

Commit message: mapping coverage

File: src/tractor_bringup/urdf/tractor.urdf.xacro (robot description, xacro)
@@ -17,4 +17,9 @@
   <xacro:property name="platform_height" value="0.0025"/> <!-- 2.5mm -->
   <xacro:property name="platform_offset_z" value="0.05"/>  <!-- 50mm -->
+  <!-- Downward pitch of the RealSense (radians, +ve tilts the lens toward the
+       ground). Keep this matched to the PHYSICAL mount. 0 = level. A small
+       downward tilt (~0.087-0.17 rad = 5-10deg) lets the depth camera see the
+       near ground plane and low obstacles for the costmap. -->
+  <xacro:property name="camera_pitch" value="0.0"/>
   <!-- Materials -->
   <material name="red">
@@ -314,5 +319,6 @@
     <!-- Camera mount tower raised 175mm: optical center now 186.5 + 175 = 361.5mm from ground -->
     <!-- Platform at 109.25mm, so offset = 361.5 - 109.25 = 252.25mm -->
-    <origin xyz="0.12085 0 0.25225" rpy="0 0 0"/>
+    <!-- camera_pitch tilts the lens down; keep matched to the physical mount. -->
+    <origin xyz="0.12085 0 0.25225" rpy="0 ${camera_pitch} 0"/>
   </joint>
   <!-- GPS Joint REMOVED -->
